File: ZoeaL/ZoeaL.kicad_pcb (KiCad board)
At the start: 2 copper layers, 100 x 57.7 mm, 44 parts, among them J1 USB_C_Receptacle_USB2.0, J2 USB_C_Receptacle_USB2.0, J3 Conn_01x06, SW11 SW_ChocV2, SW12 SW_ChocV2, SW13 SW_ChocV2, SW14 SW_ChocV2, U1 STM32F042K6Tx, U2 AP7333

Commit message: wiring angle
Parts:
- moved D11 4.79 mm to (82.5, 23.6)
- moved D12 4.77 mm to (63.5, 14.0)
- moved D13 4.77 mm to (44.5, 14.0)
- moved D14 4.72 mm to (24.4, 16.2)
- moved R1 4.20 mm to (39.2, 35.5)
- moved R11 1.98 mm to (16.5, 11.5)
- moved R12 1.98 mm to (16.2, 9.49)
- moved C11 1.98 mm to (16.9, 13.4)
- moved L11 0.40 mm to (87.3, 26.9)
- moved L13 0.40 mm to (49.5, 17.0)
- moved L14 0.40 mm to (29.8, 18.3)
- moved SW13 0.40 mm to (49.5, 12.0)
- moved SW14 0.40 mm to (29.0, 13.4)
- moved D0 0.40 mm to (78.0, 30.4)
- moved L12 0.40 mm to (68.5, 17.0)
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Routing:
- net ROW3: track 19.1 -> 12.3 mm
- net ROW4: track 36.0 -> 29.6 mm
- net Net-(D0-Pad1): track 8.23 -> 11.4 mm
- net ROW1: track 30.6 -> 33.5 mm
- net VCC: track 109.8 -> 107.5 mm
- net Net-(RB1-Pad1): track 13.0 -> 15.0 mm
- net Net-(D1-Pad1): track 2.00 -> 0.00 mm
- net COL1: track 45.7 -> 43.9 mm
- net ROW2: track 21.0 -> 19.8 mm
- net Net-(D11-Pad1): track 3.02 -> 4.02 mm
- net Net-(D14-Pad1): track 3.02 -> 4.02 mm
- net Net-(D13-Pad1): track 3.03 -> 4.03 mm
- net Net-(D12-Pad1): track 3.03 -> 4.03 mm
Other:
- board size 100 x 57.7 mm -> 99.6 x 57.7 mm

Commit message: 200904 for submit
Parts:
- added CL11: 0.1uF, Capacitor_SMD:C_0805_2012Metric_Pad1.15x1.40mm_HandSolder, F.Cu at (87.1, 29.4)
- added CL12: 0.1uF, Capacitor_SMD:C_0805_2012Metric_Pad1.15x1.40mm_HandSolder, F.Cu at (68.5, 19.5)
- added CL13: 0.1uF, Capacitor_SMD:C_0805_2012Metric_Pad1.15x1.40mm_HandSolder, F.Cu at (49.5, 19.5)
- added CL14: 0.1uF, Capacitor_SMD:C_0805_2012Metric_Pad1.15x1.40mm_HandSolder, F.Cu at (30.2, 20.8)
- added CLB1: 0.1uF, Capacitor_SMD:C_0805_2012Metric_Pad1.15x1.40mm_HandSolder, F.Cu at (17.8, 50.5)
- L11, L12, L13, L14, LB1: value LC8822 -> SK6812-MINI-E; footprint key-parts:LC8822 -> key-parts:SK6812-MINI-E
- moved D13 13.7 mm to (58.1, 12.6)
- moved D14 13.7 mm to (37.6, 12.6)
- moved D0 7.08 mm to (73.0, 25.4), turned to 180 degrees
- moved R1 6.12 mm to (42.3, 30.2), turned to 180 degrees
- moved J3 4.25 mm to (44.7, 37.2)
- moved D1 3.94 mm to (40.7, 37.3), turned to 180 degrees
- moved D11 3.86 mm to (79.0, 22.0)
- moved D12 3.86 mm to (59.9, 12.6)
- moved C6 2.53 mm to (42.3, 32.2)
- moved R11 2.40 mm to (18.9, 11.1)
- moved R12 2.40 mm to (18.6, 9.11)
- moved CB1 2.40 mm to (22.9, 36.5)
- moved RB2 2.40 mm to (21.6, 32.7)
- moved RB1 2.40 mm to (22.2, 34.6)
- moved C11 2.40 mm to (19.2, 13.1)
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Connections:
- net Net-(D0-Pad1) renamed 4V3
- D1 pad 1: Net-(D1-Pad1) -> GND
- D1 pad 2: LED -> Net-(D1-Pad2)
- J1 pad B8: LCO -> LDO
- L11 pad 3: Net-(L11-Pad3) -> GND
- L12 pad 3: Net-(L12-Pad3) -> GND
- L12 pad 4: Net-(L11-Pad3) -> Net-(L11-Pad2)
- L13 pad 3: Net-(L13-Pad3) -> GND
- L13 pad 4: Net-(L12-Pad3) -> Net-(L12-Pad2)
- L14 pad 3: Net-(L14-Pad3) -> GND
- L14 pad 4: Net-(L13-Pad3) -> Net-(L13-Pad2)
- LB1 pad 2: LCO -> LDO
- LB1 pad 3: LDO -> GND
- LB1 pad 4: Net-(L14-Pad3) -> Net-(L14-Pad2)
- R1 pad 1: Net-(D1-Pad1) -> LED
- R1 pad 2: GND -> Net-(D1-Pad2)
- U1 pad 11: LCI -> (no net)
- U1 pad 12: (no net) -> LDI
- U1 pad 13: LDI -> (no net)
Routing:
- net LCI: track 58.4 -> 0.00 mm, vias 1 -> 0
- net Net-(L14-Pad3): track 35.8 -> 0.00 mm
- net LCO: track 35.5 -> 0.00 mm, vias 1 -> 0
- net GND: track 79.0 -> 109.5 mm
- net Net-(L11-Pad3): track 21.4 -> 0.00 mm
- net 5V: track 159.2 -> 178.8 mm, vias 5 -> 9
- net Net-(L13-Pad3): track 17.8 -> 0.00 mm
- net Net-(L12-Pad3): track 17.0 -> 0.00 mm
- net LDI: track 58.9 -> 46.5 mm, vias 1 -> 2
- net Net-(D14-Pad1): track 4.02 -> 15.8 mm
- net Net-(D13-Pad1): track 4.03 -> 15.8 mm
- net ROW4: track 29.6 -> 18.8 mm
- net NRST: track 13.3 -> 21.5 mm
- net Net-(D1-Pad2): track 0.00 -> 8.21 mm
- net LED: track 9.73 -> 2.41 mm
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Other:
- outline, holes or cut-outs redrawn
- board text added: "CLK"
- board text added: "DIO"
- board text added: "GND"
- board text added: "RX"
- board text added: "TX"
- board text added: "ZoeaL by orihikarna 20/09/04"
- board text added: "nRST"
